Commit message: Updated Robot Urdf/Xacro

File: src/mobile_robot/urdf/robot.urdf.xacro (robot description, xacro)
@@ -83,13 +83,4 @@
     </joint>
   </xacro:macro>
-  <!-- ========================= -->
-  <!-- World                     -->
-  <!-- ========================= -->
-  <link name="world"/>
-  <joint name="world_to_base_link" type="fixed">
-    <parent link="world"/>
-    <child link="base_link"/>
-    <origin xyz="0 0 ${base_height / 2.0}" rpy="0 0 0"/>
-  </joint>
   <!-- ========================= -->
   <!-- Base                      -->
@@ -180,3 +171,22 @@
     <origin xyz="${lidar_x} 0 ${lidar_z}" rpy="0 0 0"/>
   </joint>
+  <!-- ========================= -->
+  <!-- Gazebo Diff Drive         -->
+  <!-- ========================= -->
+  <gazebo>
+    <plugin
+      filename="gz-sim-diff-drive-system"
+      name="gz::sim::systems::DiffDrive">
+      <left_joint>left_wheel_joint</left_joint>
+      <right_joint>right_wheel_joint</right_joint>
+      <wheel_separation>${2.0 * wheel_y}</wheel_separation>
+      <wheel_radius>${wheel_radius}</wheel_radius>
+      <topic>/cmd_vel</topic>
+      <odom_topic>/odom</odom_topic>
+      <tf_topic>/tf</tf_topic>
+      <frame_id>odom</frame_id>
+      <child_frame_id>base_link</child_frame_id>
+      <odom_publish_frequency>30</odom_publish_frequency>
+    </plugin>
+  </gazebo>
 </robot>

Commit message: added IMU sensor

File: src/mobile_robot/urdf/robot.urdf.xacro (robot description, xacro)
@@ -222,3 +222,27 @@
     </sensor>
   </gazebo>
+  <!-- ========================= -->
+  <!-- IMU                       -->
+  <!-- ========================= -->
+  <link name="imu_link">
+    <visual>
+      <geometry>
+        <box size="0.08 0.08 0.03"/>
+      </geometry>
+      <material name="gray"/>
+    </visual>
+  </link>
+  <joint name="imu_joint" type="fixed">
+    <parent link="base_link"/>
+    <child link="imu_link"/>
+    <origin xyz="0 0 0.13" rpy="0 0 0"/>
+  </joint>
+  <gazebo reference="imu_link">
+    <sensor name="imu_sensor" type="imu">
+      <pose>0 0 0 0 0 0</pose>
+      <always_on>true</always_on>
+      <update_rate>50</update_rate>
+      <topic>/imu</topic>
+    </sensor>
+  </gazebo>
 </robot>
