Commit message: Create Mission BT package with BehaviorTree.CPP integration

File: src/mobile_robot/urdf/robot.urdf.xacro (robot description, xacro)
@@ -13,4 +13,5 @@
   <xacro:property name="wheel_y"      value="0.29"/>
   <xacro:property name="wheel_z"      value="-0.05"/>
+  <xacro:property name="wheel_x"      value="0.0"/>
   <xacro:property name="caster_radius" value="0.08"/>
   <xacro:property name="caster_x"      value="-0.35"/>
@@ -79,5 +80,5 @@
       <parent link="base_link"/>
       <child link="${prefix}_wheel_link"/>
-      <origin xyz="0 ${y} ${wheel_z}" rpy="0 0 0"/>
+      <origin xyz="${wheel_x} ${y} ${wheel_z}" rpy="0 0 0"/>
       <axis xyz="0 1 0"/>
     </joint>

Commit message: added wait action

File: src/mobile_robot/urdf/robot.urdf.xacro (robot description, xacro)
@@ -14,4 +14,7 @@
   <xacro:property name="wheel_z"      value="-0.05"/>
   <xacro:property name="wheel_x"      value="0.0"/>
+  <xacro:property name="front_caster_radius" value="0.04"/>
+  <xacro:property name="front_caster_x" value="0.45"/>
+  <xacro:property name="front_caster_z" value="-0.1"/>
   <xacro:property name="caster_radius" value="0.08"/>
   <xacro:property name="caster_x"      value="-0.35"/>
@@ -141,4 +144,46 @@
     <origin xyz="${caster_x} 0 ${caster_z}" rpy="0 0 0"/>
   </joint>
+  <link name="front_support_link">
+    <visual>
+      <geometry>
+        <sphere radius="${front_caster_radius}"/>
+      </geometry>
+      <material name="gray"/>
+    </visual>
+    <collision>
+      <geometry>
+        <sphere radius="${front_caster_radius}"/>
+      </geometry>
+    </collision>
+    <inertial>
+      <mass value="0.05"/>
+      <inertia
+        ixx="0.00003"
+        ixy="0.0"
+        ixz="0.0"
+        iyy="0.00003"
+        iyz="0.0"
+        izz="0.00003"/>
+    </inertial>
+  </link>
+  <joint name="front_support_joint" type="fixed">
+    <parent link="base_link"/>
+    <child link="front_support_link"/>
+    <origin
+      xyz="${front_caster_x} 0 ${front_caster_z}"
+      rpy="0 0 0"/>
+  </joint>
+  <gazebo reference="front_support_link">
+    <mu1>0.01</mu1>
+    <mu2>0.01</mu2>
+  </gazebo>
+  <gazebo reference="left_wheel_link">
+    <mu1>1.2</mu1>
+    <mu2>1.2</mu2>
+  </gazebo>
+  <gazebo reference="right_wheel_link">
+    <mu1>1.2</mu1>
+    <mu2>1.2</mu2>
+  </gazebo>
   <!-- ========================= -->
   <!-- Lidar                     -->

Commit message: improvements

File: src/mobile_robot/urdf/robot.urdf.xacro (robot description, xacro)
@@ -139,8 +139,10 @@
     </inertial>
   </link>
-  <joint name="caster_wheel_joint" type="fixed">
+  <joint name="caster_wheel_joint" type="continuous">
     <parent link="base_link"/>
     <child link="caster_wheel_link"/>
     <origin xyz="${caster_x} 0 ${caster_z}" rpy="0 0 0"/>
+    <axis xyz="0 0 1"/>
+    <dynamics damping="0.0" friction="0.0"/>
   </joint>
   <link name="front_support_link">
@@ -167,5 +169,5 @@
     </inertial>
   </link>
-  <joint name="front_support_joint" type="fixed">
+  <joint name="front_support_joint" type="continuous">
     <parent link="base_link"/>
     <child link="front_support_link"/>
@@ -173,4 +175,6 @@
       xyz="${front_caster_x} 0 ${front_caster_z}"
       rpy="0 0 0"/>
+    <axis xyz="0 0 1"/>
+    <dynamics damping="0.0" friction="0.0"/>
   </joint>
   <gazebo reference="front_support_link">
